File: hw/orbtrace_m26/orbtrace_m26/USB.kicad_sch (KiCad schematic)
At the start: 63 parts, among them J1 USB_C_Receptacle_USB2.0_16P, SW1 SW_Push_Shielded, U1 USB3343, U2 USBLC6-2P6, U3 TLV71325PDQN, U4 TLV62568PDRL, U5 TLV62568PDRL

Commit message: Init PCB without error
Connections:
- net GND: now also U3.5 (PAD); no longer U3.PAD
Changed lines of the file:
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@@
 	(title_block
 		(title "Orbtrace m26")
-		(date "2026-08-04")
-		(rev "draft")
+		(date "2026-08-11")
+		(rev "Run 1")
 		(comment 1 "${SHEETNAME}")
 	)
@@
 			)
 		)
-		(pin "PAD"
+		(pin "5"
 		)
 		(pin "4"
