File: hw/orbtrace_m26/orbtrace_m26/FPGA.kicad_sch (KiCad schematic)
At the start: 81 parts, among them J2 Conn_01x05, U6 LFE5U-25F-6BG256C, U7 M24128-BFMH, U8 W956A8MBYA5I, U9 S25FL064LABBHV020, Y1 831025497

Commit message: Init PCB without error
Connections:
- new net: U9.A2 (NC), U9.A3 (NC), U9.A5 (NC), U9.B5 (NC), U9.C5 (NC), U9.D5 (NC), U9.E1 (NC), U9.E2 (NC), U9.E3 (NC), U9.E4 (NC), U9.E5 (NC)
- new net: U9.B1 (DNU), U9.C1 (DNU), U9.D1 (DNU)
Changed lines of the file:
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@@
 	(title_block
 		(title "Orbtrace m26")
-		(date "2026-08-04")
-		(rev "draft")
+		(date "2026-08-11")
+		(rev "Run 1")
 		(comment 1 "${SHEETNAME}")
 	)
@@
 		(pin "D4"
 		)
+		(pin "A5"
+		)
+		(pin "A2"
+		)
+		(pin "C2"
+		)
 		(instances
 			(project "orbtrace_m26"
@@
 		(pin "A4"
 		)
+		(pin "A3"
+		)
+		(pin "E4"
+		)
+		(pin "D5"
+		)
+		(pin "D1"
+		)
+		(pin "E2"
+		)
+		(pin "C1"
+		)
+		(pin "E3"
+		)
+		(pin "E1"
+		)
+		(pin "E5"
+		)
+		(pin "C3"
+		)
+		(pin "A5"
+		)
+		(pin "B5"
+		)
+		(pin "A2"
+		)
+		(pin "C5"
+		)
+		(pin "B1"
+		)
 		(instances

Commit message: WIP on PCB
Parts:
- added R68, R69, R70, R71, R72, R73, R74, R75, R76, R77, R78, R79, R80, R81, R82, R83, R84, R85, R86: 0Ω, Resistor_SMD:R_0402_1005Metric, symbol orbtrace:R
Connections:
- net HRAM_CLK: now also R77.1; no longer TP46.1
- net HRAM_CS: now also R76.1; no longer TP42.1
- net HRAM_DQ0: now also R78.1; no longer TP26.1
- net HRAM_DQ1: now also R79.1; no longer TP27.1
- net HRAM_DQ2: now also R80.1; no longer TP29.1
- net HRAM_DQ3: now also R81.1; no longer TP31.1
- net HRAM_DQ4: now also R82.1; no longer TP35.1
- net HRAM_DQ5: now also R83.1; no longer TP39.1
- net HRAM_DQ6: now also R84.1; no longer TP43.1
- net HRAM_DQ7: now also R85.1; no longer TP47.1
- net HRAM_RST: now also R74.1; no longer TP34.1
- net HRAM_RWDS: now also R75.1; no longer TP38.1
- net QSPI_CS: now also R73.1; no longer TP45.1
- net QSPI_IO0: now also R68.1; no longer TP28.1
- net QSPI_IO1: now also R69.1; no longer TP30.1
- net QSPI_IO2: now also R70.1; no longer TP33.1
- net QSPI_IO3: now also R71.1; no longer TP37.1
- net QSPI_SCK: now also R72.1; no longer TP41.1
- net SYS_CLK: now also R86.1; no longer TP23.1
- new net: R71.2, TP37.1
- new net: R77.2, TP46.1
- new net: R84.2, TP43.1
- new net: R76.2, TP42.1
- new net: R70.2, TP33.1
- new net: R72.2, TP41.1
- new net: R81.2, TP31.1
- new net: R80.2, TP29.1
- new net: R83.2, TP39.1
- new net: R82.2, TP35.1
- new net: R85.2, TP47.1
- new net: R78.2, TP26.1
- new net: R86.2, TP23.1
- new net: R75.2, TP38.1
- new net: R74.2, TP34.1
- new net: R69.2, TP30.1
- new net: R79.2, TP27.1
- new net: R73.2, TP45.1
- new net: R68.2, TP28.1
Other:
- moved on the sheet: TP23, TP26, TP27, TP28, TP29, TP30, TP31, TP33, TP34, TP35, TP37, TP38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
