File: hw/orbtrace_m26/orbtrace_m26/usb.kicad_sch (KiCad schematic)
At the start: 64 parts, among them J1 USB_C_Receptacle_USB2.0_16P, SW1 SW_Push_Shielded, U1 USB3343, U2 USBLC6-2P6, U3 TLV71325PDQN, U4 TLV62568PDRL, U5 TLV62568PDRL

Commit message: WIP on PCB
Parts:
- removed C10, C9: 10µF, Capacitor_SMD:C_0603_1608Metric, symbol orbtrace:C
- removed C15: 22µF, Capacitor_SMD:C_0805_2012Metric, symbol orbtrace:C
- removed R1: 10k, Resistor_SMD:R_0402_1005Metric, symbol orbtrace:R
- removed R10, R13: 475k, Resistor_SMD:R_0402_1005Metric, symbol orbtrace:R
- removed R11: 100k, Resistor_SMD:R_0402_1005Metric, symbol orbtrace:R
- removed R9: 453k, Resistor_SMD:R_0402_1005Metric, symbol orbtrace:R
- removed SW1: SW_Push_Shielded, orbtrace:SW_Wurth_WS-TASV_435151014824, symbol orbtrace:SW_Push_Shielded
- removed TP1, TP10, TP100, TP11, TP12, TP13, TP14, TP15, TP16, TP17, TP18, TP19, TP2, TP20, TP21, TP3, TP4, TP5, TP6, TP7, TP8, TP9: (no value), TestPoint:TestPoint_Pad_D1.0mm, symbol orbtrace:TestPoint_Flag
- removed U4, U5: TLV62568PDRL, Package_TO_SOT_SMD:SOT-563, symbol orbtrace:TLV62568PDRL
- added R7: 210k, symbol orbtrace:R
- added R8: 47k, symbol orbtrace:R
- added U3, U5: TLV62569DRL, symbol orbtrace:TLV62569DRL
- C1: footprint Capacitor_SMD:C_0402_1005Metric -> (none); Dielectric X7S -> X7R; Internal reference C_002 -> (none); Voltage rating DC 16 V -> 10 V
- C10: renamed from C13; footprint Capacitor_SMD:C_0603_1608Metric -> (none); Internal reference C_006 -> (none)
- C11: renamed from C12; footprint Capacitor_SMD:C_0402_1005Metric -> (none); Dielectric C0G -> X7R; Internal reference C_005 -> (none); Tolerance 0.1 pF -> 10 %; Voltage rating DC 50 V -> 6.3 V
- C12: renamed from C14; footprint Capacitor_SMD:C_0805_2012Metric -> (none); Internal reference C_004 -> (none); Package 0805 -> 0603; Tolerance 20 % -> 10 %; Voltage rating DC 6.3 V -> 4 V
- C13: renamed from C16; footprint Capacitor_SMD:C_0805_2012Metric -> (none); Internal reference C_004 -> (none); Package 0805 -> 0603; Tolerance 20 % -> 10 %; Voltage rating DC 6.3 V -> 4 V
- C14: renamed from C17; footprint Capacitor_SMD:C_0402_1005Metric -> (none); Internal reference C_002 -> (none); Voltage rating DC 16 V -> 4 V
- C2: footprint Capacitor_SMD:C_0402_1005Metric -> (none); Internal reference C_002 -> (none); Voltage rating DC 16 V -> 4 V
- C3, C4: footprint Capacitor_SMD:C_0402_1005Metric -> (none); Internal reference C_003 -> (none); Voltage rating DC 16 V -> 10 V
- C5: footprint Capacitor_SMD:C_0805_2012Metric -> (none); Internal reference C_007 -> (none); Voltage rating DC 500 V -> 250 V
- C6: renamed from C7; footprint Capacitor_SMD:C_0603_1608Metric -> (none); Internal reference C_006 -> (none)
- C7: renamed from C6; footprint Capacitor_SMD:C_0402_1005Metric -> (none); Dielectric C0G -> X7R; Internal reference C_005 -> (none); Tolerance 0.1 pF -> 10 %; Voltage rating DC 50 V -> 10 V
- C8: footprint Capacitor_SMD:C_0603_1608Metric -> (none); Dielectric X7T -> X7R; Internal reference C_001 -> (none); Tolerance 20 % -> 10 %
- C9: renamed from C11; footprint Capacitor_SMD:C_0402_1005Metric -> (none); Dielectric X7S -> X7R; Internal reference C_002 -> (none); Voltage rating DC 16 V -> 10 V
- D1: footprint LED_SMD:LED_0603_1608Metric -> (none); Forward Voltage 3.2 V -> 2.85 V; Internal reference D_003 -> (none)
- F1: footprint Fuse:Fuse_0805_2012Metric -> (none); Internal reference F_001 -> (none)
- J1: Internal reference J_006 -> (none)
- L1, L2: footprint Inductor_SMD:L_1210_3225Metric_Pad1.42x2.65mm_HandSolder -> (none); DCR R: 43 mΩ -> R: __; I rms / DC I_{rms}: 2.9 A -> I_{rms}: __ mA; I sat I_{sat}: 4 A -> I_{sat}: __ mA; Internal reference L_002 -> (none); Package 1210 -> 0805; SRF SRF: 35 MHz -> SRF: __ MHz
- R1: renamed from R2; footprint Resistor_SMD:R_0402_1005Metric -> (none); Internal reference R_012 -> (none)
- R10: renamed from R14; footprint Resistor_SMD:R_0402_1005Metric -> (none); Internal reference R_004 -> (none)
- R11: renamed from R3; value 180Ω -> 27k; footprint Resistor_SMD:R_0402_1005Metric -> (none); Internal reference R_011 -> (none); Package 0402 -> 0603; Power 1/16 W -> 1/10 W
- R2: renamed from R4; footprint Resistor_SMD:R_0402_1005Metric -> (none); Internal reference R_013 -> (none)
- R3: renamed from R5; footprint Resistor_SMD:R_0402_1005Metric -> (none); Internal reference R_014 -> (none)
- R4: renamed from R6; footprint Resistor_SMD:R_0402_1005Metric -> (none); Internal reference R_009 -> (none); Power 1/16 W -> 1/10 W
- R5: renamed from R7; footprint Resistor_SMD:R_0402_1005Metric -> (none); Internal reference R_009 -> (none); Power 1/16 W -> 1/10 W
- R6: renamed from R8; footprint Resistor_SMD:R_0402_1005Metric -> (none); Internal reference R_010 -> (none); Package 0402 -> 1206; Power 1/16 W -> 1/4 W; Temp coef 100 ppm -> 200 ppm; Tolerance 1% -> 5 %
- R9: renamed from R12; value 82.5k -> 84.5k; footprint Resistor_SMD:R_0402_1005Metric -> (none); Internal reference R_008 -> (none)
- U1: Internal reference U_008 -> (none)
- U2: footprint Package_TO_SOT_SMD:SOT-666 -> (none); Internal reference D_002 -> (none)
- U4: renamed from U3; footprint orbtrace:Texas_X2SON-4_1x1mm_P0.65mm -> (none); Internal reference U_010 -> (none); Package X2SON-4 -> (none)
Connections:
- net +3.3V: now also R7.2
- net +5V: now also U3.3 (VIN), U3.5 (EN), U5.3 (VIN), U5.5 (EN)
- net GND: now also U4.PAD, R8.1, U3.2 (GND), U5.2 (GND); no longer U4.5 (PAD)
- net at L1.1: now also U3.4 (SW)
- net at C7.2: now also R7.1, R8.2, U3.1 (FB)
- net at C11.2, R10.2, R9.1: now also U5.1 (FB)
- net at L2.1: now also U5.4 (SW)
- net VBUS: no longer names the net of F1.2, J1.A4 (VBUS), J1.A9 (VBUS), J1.B4 (VBUS), J1.B9 (VBUS)
Other:
- note added: "Warning: If = 0.08mA ~ 0.1 mA with Vf = 2.3"
- note removed: ".8-pF capacitance is recommended for R2 of 100-kΩ resistance."
- note removed: "Button"
- note removed: "I_{F}: 10mA (nom. 20mA), V_{F} = 3.2V R = (5-3.2)/0.01 = 180R"
- note removed: "LED POWER"
- note removed: "Pour V_{S} = 1.1V, (R_{1} / R_{2}) = 5/6"
- note removed: "Pour V_{S} = 3.3V, (R_{1} / R_{2}) = 9/2"
- note removed: "V_{s} = V_{FB} x (1 + R_{1} / R_{2}) V_{FB} typ.: 0.6V (R_{1} / R_{2}) = (V_{s} / V_{FB}) - 1"
- moved on the sheet: C10, C11, C12, C13, C14, C6, C7, C8, D1, L1, L2, R10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
