File: hw/orbtrace_m26/orbtrace_m26/JTAG.kicad_sch (KiCad schematic)
At the start: 110 parts, among them J3 Conn_01x08, J4 Conn_01x08, U10 SWD-TRACE-FTSH110, U11 SN74AVC4T774-Q1, U12 SN74AVC4T774-Q1, U13 SWD-FTSH105, U14 SN74AVC4T774-Q1, U15 SN74AVC4T774-Q1, U16 TLA2024

Commit message: WIP on PCB
Parts:
- added TP101, TP102, TP103: (no value), TestPoint:TestPoint_Pad_D1.0mm, symbol orbtrace:TestPoint_Flag
Connections:
- net GND: now also TP101.1, TP102.1
- net at C54.1, FB2.1, U10.1 (VTREF): now also TP103.1
- net at C59.1, FB3.2, U13.1 (VTREF): no longer TP49.1
- net at C60.1, FB4.2, J3.1 (Pin_1): now also TP49.1

Commit message: WIP
Parts:
- TP50, TP51, TP54, TP55, TP57, TP58, TP60, TP61, TP63, TP64, TP66, TP67, TP70, TP73, TP74, TP77, TP78, TP81, TP82, TP85, TP86, TP88, TP89, TP90, TP91, TP92: now not fitted
Connections:
- net DEBUG_JTCK: now also U11.5 (A3); no longer U11.3 (A1)
- net DEBUG_JTDI: now also U11.3 (A1); no longer U11.5 (A3)
- net DEBUG_JTDO: now also U11.4 (A2); no longer U11.6 (A4)
- net DEBUG_JTMS: now also U11.6 (A4); no longer U11.4 (A2)
- net DEBUG_NRST: now also U14.6 (A4); no longer U14.4 (A2)
- net DIR_JTCK: now also U11.7 (DIR3); no longer U11.1 (DIR1)
- net DIR_JTDI: now also U11.1 (DIR1); no longer U11.7 (DIR3)
- net DIR_JTMS: now also U11.8 (DIR4); no longer U11.2 (DIR2)
- net DIR_NRST: now also U14.8 (DIR4); no longer U14.2 (DIR2)
- net GND: now also U11.2 (DIR2), U12.7 (DIR3), U12.8 (DIR4), U14.2 (DIR2); no longer U11.8 (DIR4), U12.1 (DIR1), U12.2 (DIR2), U14.8 (DIR4)
- net SPARE_DIR0: now also U15.1 (DIR1); no longer U15.7 (DIR3)
- net SPARE_DIR1: now also U15.2 (DIR2); no longer U15.8 (DIR4)
- net SPARE_DIR2: now also U15.7 (DIR3); no longer U15.1 (DIR1)
- net SPARE_DIR3: now also U15.8 (DIR4); no longer U15.2 (DIR2)
- net SPARE_DIR4: now also U12.1 (DIR1); no longer U12.7 (DIR3)
- net SPARE_DIR5: now also U12.2 (DIR2); no longer U12.8 (DIR4)
- net SPARE_IO0: now also U15.3 (A1); no longer U15.5 (A3)
- net SPARE_IO1: now also U15.4 (A2); no longer U15.6 (A4)
- net SPARE_IO2: now also U15.5 (A3); no longer U15.3 (A1)
- net SPARE_IO3: now also U15.6 (A4); no longer U15.4 (A2)
- net SPARE_IO4: now also U12.3 (A1); no longer U12.5 (A3)
- net SPARE_IO5: now also U12.4 (A2); no longer U12.6 (A4)
- net TRACE_CLK: now also U14.5 (A3); no longer U14.3 (A1)
- net TRACE_D0: now also U14.4 (A2); no longer U14.6 (A4)
- net TRACE_D1: now also U14.3 (A1); no longer U14.5 (A3)
- net TRACE_D2: now also U12.6 (A4); no longer U12.4 (A2)
- net TRACE_D3: now also U12.5 (A3); no longer U12.3 (A1)
- net at R37.1: now also U12.13 (B2); no longer U12.11 (B4)
- net at R50.1: now also U14.13 (B2); no longer U14.11 (B4)
- net at R30.1: now also U11.12 (B3); no longer U11.14 (B1)
- net at U14.12 (B3): now also R42.1; no longer R47.1
- net at R45.1: now also U14.11 (B4); no longer U14.13 (B2)
- net at U14.14 (B1): now also R47.1; no longer R42.1
- net at U15.11 (B4): now also R46.1; no longer R51.1
- net at U15.12 (B3): now also R43.1; no longer R48.1
- net at U15.13 (B2): now also R51.1; no longer R46.1
- net at U15.14 (B1): now also R48.1; no longer R43.1
- net at R31.1: now also U12.12 (B3); no longer U12.14 (B1)
- net at R32.1: now also U11.11 (B4); no longer U11.13 (B2)
- net at R33.1: now also U12.11 (B4); no longer U12.13 (B2)
- net at R36.1: now also U11.13 (B2); no longer U11.11 (B4)
- net at R34.1: now also U11.14 (B1); no longer U11.12 (B3)
- net at R35.1: now also U12.14 (B1); no longer U12.12 (B3)
Other:
- note added: "Run 1: Remove from CI"
- moved on the sheet: R30, R31, R32, R33, R34, R35, R36, R37, R42, R43, R45, R46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
