File: hw/orbtrace_m26/orbtrace_m26/LEDs.kicad_sch (KiCad schematic)
At the start: 22 parts, among them U17 SN74LVC1T45DBV, U18 WL-ICLED, U19 WL-ICLED, U20 WL-ICLED, U21 WL-ICLED, U22 WL-ICLED

Commit message: WIP
Other:
- note added: "DEBUG"
- note added: "STATUS"
- note added: "TRACE"
- note added: "VTPWR"
- note added: "VTREF"
Changed lines of the file:
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@@
+		)
+	)
+	(text "VTREF"
+		(exclude_from_sim no)
+		(at 155.194 75.946 0)
+		(effects
+			(font
+				(size 1.27 1.27)
+			)
+		)
+	)
+	(text "VTPWR"
+		(exclude_from_sim no)
+		(at 180.594 76.2 0)
+		(effects
+			(font
+				(size 1.27 1.27)
+			)
+		)
+	)
+	(text "DEBUG"
+		(exclude_from_sim no)
+		(at 104.394 76.2 0)
+		(effects
+			(font
+				(size 1.27 1.27)
+			)
+		)
+	)
+	(text "STATUS"
+		(exclude_from_sim no)
+		(at 79.248 76.2 0)
+		(effects
+			(font
+				(size 1.27 1.27)
+			)
+		)
+	)
+	(text "TRACE"
+		(exclude_from_sim no)
+		(at 129.794 75.946 0)
+		(effects
+			(font
+				(size 1.27 1.27)
+			)
 		)
 	)
