File: hw/orbtrace_m26/orbtrace_m26/orbtrace_m26.kicad_pcb (KiCad board)
At the start: 4 copper layers, 13.4 x 4.5 mm, 281 parts, among them J1 USB_C_Receptacle_USB2.0_16P, J2 Conn_01x05, J3 Conn_01x08, J4 Conn_01x08, J5 Conn_02x35_Odd_Even, SW1 SW_Push_Shielded, U1 USB3343, U10 SWD-TRACE-FTSH110, U11 SN74AVC4T774-Q1, U12 SN74AVC4T774-Q1, U13 SWD-FTSH105, U14 SN74AVC4T774-Q1, U15 SN74AVC4T774-Q1, U16 TLA2024, U17 SN74LVC1T45DBV, U18 WL-ICLED, U19 WL-ICLED, U2 USBLC6-2P6, U20 WL-ICLED, U21 WL-ICLED, U22 WL-ICLED, U3 TLV71325PDQN, U4 TLV62568PDRL, U5 TLV62568PDRL, U6 LFE5U-25F-6BG256C, U7 M24128-BFMH, U8 W956A8MBYA5I, U9 S25FL064LABBHV020, Y1 831025497

Commit message: WIP on PCB
Parts:
- C1, C19, C2, C20, C21, C22, C23, C24, C25, C26, C27, C28, C29, C3, C30, C31, C32, C33, C34, C35, C36, C37, C38, C39, C4, C40, C41, C42, R5, R6, R7, TP1, TP10, TP11, TP12, TP13, TP14, TP15, TP16, TP17, TP18, TP19, TP2, TP20, TP24, TP25, TP26, TP27, TP28, TP29, TP3, TP30, TP31, TP33, TP34, TP35, TP37, TP38, TP39, TP4, TP41, TP42, TP43, TP45, TP46, TP47, TP5, TP50, TP51, TP54, TP55, TP57, TP58, TP6, TP60, TP61, TP63, TP64, TP66, TP67, TP7, TP70, TP73, TP74, TP77, TP78, TP8, TP81, TP82, TP85, TP86, TP88, TP89, TP9, TP90, TP91, TP92: moved to B.Cu
- moved TP75 218.9 mm to (256.7, 44.1)
- moved TP83 218.9 mm to (259.8, 44.1)
- moved TP68 218.8 mm to (253.7, 44.1)
- moved TP79 218.6 mm to (256.7, 47.2)
- moved TP71 218.6 mm to (253.7, 47.2)
- moved TP87 218.6 mm to (259.8, 47.2)
- moved J3 193.0 mm to (241.0, 32.0)
- moved TP8 188.5 mm to (234.8, 125.2), turned to 180 degrees
- moved C60 188.0 mm to (244.8, 33.2)
- moved R56 184.3 mm to (246.5, 39.0)
- moved R24 183.0 mm to (224.8, 68.2)
- moved R25 183.0 mm to (224.8, 70.2)
- moved R26 183.0 mm to (224.8, 72.2)
- moved FB4 182.3 mm to (245.3, 31.0)
- moved R57 182.1 mm to (246.5, 41.0)
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Routing:
- net GND: track 0.00 -> 13.5 mm, vias 0 -> 1
- net +3.3V: track 0.00 -> 10.4 mm, vias 0 -> 3
- net Net-(U4-PD): track 0.00 -> 7.24 mm, vias 0 -> 2
- net USB_D_P: track 0.00 -> 5.72 mm
- net USB_D_N: track 0.00 -> 5.34 mm
- net +5V: track 0.00 -> 4.39 mm, vias 0 -> 1
- net Net-(U4-FB): track 0.00 -> 4.03 mm
- net Net-(U1-RBIAS): track 0.00 -> 3.98 mm
- net Net-(U1-ID): track 0.00 -> 3.05 mm, vias 0 -> 1
- net Net-(U1-VBUS): track 0.00 -> 2.87 mm
- net ULPI_RESET: track 0.00 -> 2.01 mm, vias 0 -> 1
- net Net-(U1-VDD18): track 0.00 -> 1.83 mm, vias 0 -> 1
Other:
- board size 13.4 x 4.5 mm -> 50 x 100.1 mm

Commit message: WIP on PCB
Parts:
- added R68: 0Ω, Resistor_SMD:R_0402_1005Metric, F.Cu at (181.9, 85.0)
- added R69: 0Ω, Resistor_SMD:R_0402_1005Metric, F.Cu at (183.1, 85.0)
- added R70: 0Ω, Resistor_SMD:R_0402_1005Metric, F.Cu at (180.6, 85.0)
- added R71: 0Ω, Resistor_SMD:R_0402_1005Metric, F.Cu at (179.3, 85.0)
- added R72: 0Ω, Resistor_SMD:R_0402_1005Metric, F.Cu at (185.7, 85.0)
- added R73: 0Ω, Resistor_SMD:R_0402_1005Metric, F.Cu at (184.4, 85.0)
- added R74: 0Ω, Resistor_SMD:R_0402_1005Metric, F.Cu at (200.8, 88.3)
- added R75: 0Ω, Resistor_SMD:R_0402_1005Metric, F.Cu at (188.0, 88.3)
- added R76: 0Ω, Resistor_SMD:R_0402_1005Metric, F.Cu at (199.5, 88.3)
- added R77: 0Ω, Resistor_SMD:R_0402_1005Metric, F.Cu at (198.2, 88.3)
- added R78: 0Ω, Resistor_SMD:R_0402_1005Metric, F.Cu at (192.9, 85.0)
- added R79: 0Ω, Resistor_SMD:R_0402_1005Metric, F.Cu at (195.4, 85.0)
- added R80: 0Ω, Resistor_SMD:R_0402_1005Metric, F.Cu at (190.4, 85.0)
- added R81: 0Ω, Resistor_SMD:R_0402_1005Metric, F.Cu at (189.1, 84.9)
- added R82: 0Ω, Resistor_SMD:R_0402_1005Metric, F.Cu at (189.2, 88.3)
- added R83: 0Ω, Resistor_SMD:R_0402_1005Metric, F.Cu at (191.6, 85.0)
- added R84: 0Ω, Resistor_SMD:R_0402_1005Metric, F.Cu at (194.2, 85.0)
- added R85: 0Ω, Resistor_SMD:R_0402_1005Metric, F.Cu at (196.7, 85.0)
- added R86: 0Ω, Resistor_SMD:R_0402_1005Metric, F.Cu at (194.5, 76.4)
- added TP100: ~, TestPoint:TestPoint_Pad_D1.0mm, F.Cu at (127.2, 106.8)
- added TP101: ~, TestPoint:TestPoint_Pad_D1.0mm, B.Cu at (197.8, 41.3)
- added TP102: ~, TestPoint:TestPoint_Pad_D1.0mm, F.Cu at (122.1, 109.8)
- added TP103: ~, TestPoint:TestPoint_Pad_D1.0mm, B.Cu at (196.5, 43.2)
- C46, C47, C48, C49, R38, R39, R40, R41, R44, R49, R52, R53, R54, R55, TP23, TP52, TP53, TP56, TP59, TP62, TP65, TP69, TP72, TP76, TP80, TP84, U3: moved to B.Cu
- moved C60 111.9 mm to (132.8, 34.3)
- moved FB4 111.9 mm to (133.4, 32.0)
- moved R56 111.9 mm to (134.6, 40.1)
- moved R57 111.9 mm to (134.6, 42.0)
- moved R58 111.9 mm to (134.6, 44.0)
- moved R59 111.9 mm to (134.6, 46.0)
- moved R60 111.9 mm to (134.6, 48.0)
- moved R61 111.9 mm to (134.6, 50.0)
- moved TP75 111.9 mm to (144.8, 45.2)
- moved TP79 111.9 mm to (144.8, 48.3)
- moved J3 111.9 mm to (129.1, 33.1)
- moved TP68 111.9 mm to (141.8, 45.2)
- moved TP71 111.9 mm to (141.8, 48.3)
- moved TP83 111.9 mm to (147.8, 45.2)
- moved TP87 111.9 mm to (147.8, 48.3)
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Connections:
- TP23 pad 1: SYS_CLK -> Net-(R86-Pad2)
- TP26 pad 1: HRAM_DQ0 -> Net-(R78-Pad2)
- TP27 pad 1: HRAM_DQ1 -> Net-(R79-Pad2)
- TP28 pad 1: QSPI_IO0 -> Net-(R68-Pad2)
- TP29 pad 1: HRAM_DQ2 -> Net-(R80-Pad2)
- TP30 pad 1: QSPI_IO1 -> Net-(R69-Pad2)
- TP31 pad 1: HRAM_DQ3 -> Net-(R81-Pad2)
- TP33 pad 1: QSPI_IO2 -> Net-(R70-Pad2)
- TP34 pad 1: HRAM_RST -> Net-(R74-Pad2)
- TP35 pad 1: HRAM_DQ4 -> Net-(R82-Pad2)
- TP37 pad 1: QSPI_IO3 -> Net-(R71-Pad2)
- TP38 pad 1: HRAM_RWDS -> Net-(R75-Pad2)
- TP39 pad 1: HRAM_DQ5 -> Net-(R83-Pad2)
- TP41 pad 1: QSPI_SCK -> Net-(R72-Pad2)
- TP42 pad 1: HRAM_CS -> Net-(R76-Pad2)
- TP43 pad 1: HRAM_DQ6 -> Net-(R84-Pad2)
- TP45 pad 1: QSPI_CS -> Net-(R73-Pad2)
- TP46 pad 1: HRAM_CLK -> Net-(R77-Pad2)
- TP47 pad 1: HRAM_DQ7 -> Net-(R85-Pad2)
- TP49 pad 1: Net-(U13-VTREF) -> Net-(J3-Pin_1)
Routing:
- net VTREF: track 0.00 -> 20.3 mm, vias 0 -> 1
- net HRAM_RST: track 0.00 -> 12.6 mm
- net QSPI_SCK: track 0.00 -> 10.6 mm
- net HRAM_CS: track 0.00 -> 9.98 mm
- net HRAM_RWDS: track 0.00 -> 9.08 mm
- net HRAM_DQ2: track 0.00 -> 8.49 mm
- net QSPI_CS: track 0.00 -> 8.46 mm
- net QSPI_IO2: track 0.00 -> 7.76 mm
- net HRAM_CLK: track 0.00 -> 7.61 mm
- net HRAM_DQ3: track 0.00 -> 7.60 mm
- net VT_TRACE_D3: track 0.00 -> 7.08 mm, vias 0 -> 1
- net VT_TRACE_CLK: track 0.00 -> 7.06 mm, vias 0 -> 1
- net VT_DEBUG_JTDI: track 0.00 -> 7.06 mm, vias 0 -> 1
- net VT_DEBUG_JTCK: track 0.00 -> 7.05 mm, vias 0 -> 1
- net VT_TRACE_D1: track 0.00 -> 7.05 mm, vias 0 -> 1
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
Commit message: WIP
Parts:
- U3: moved to F.Cu
- moved TP45 26.6 mm to (183.1, 82.4)
- moved TP41 25.7 mm to (185.7, 82.4)
- moved TP37 24.0 mm to (180.6, 82.4)
- moved TP30 20.8 mm to (181.9, 85.2)
- moved TP28 19.1 mm to (184.4, 85.2)
- moved C19 19.0 mm to (174.5, 67.0)
- moved C20 19.0 mm to (164.0, 63.2)
- moved C21 19.0 mm to (170.5, 71.5)
- moved C22 19.0 mm to (165.8, 64.5)
- moved C23 19.0 mm to (165.8, 63.5)
- moved C24 19.0 mm to (169.5, 66.0)
- moved C25 19.0 mm to (168.8, 69.5)
- moved C26 19.0 mm to (169.8, 69.5)
- moved C27 19.0 mm to (170.8, 69.5)
- moved C28 19.0 mm to (173.8, 63.5)
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Routing:
- net GND: track 13.5 -> 47.9 mm, vias 1 -> 27
- net HRAM_DQ6: track 1.53 -> 20.1 mm
- net +2V5: track 0.00 -> 16.8 mm, vias 0 -> 3
- net +3.3V: track 10.4 -> 25.6 mm, vias 3 -> 13
- net HRAM_DQ4: track 5.17 -> 20.2 mm
- net HRAM_CS: track 9.98 -> 24.6 mm
- net HRAM_DQ7: track 5.72 -> 20.2 mm
- net HRAM_RST: track 12.6 -> 26.9 mm
- net HRAM_DQ5: track 5.94 -> 20.1 mm
- net HRAM_DQ1: track 6.43 -> 20.2 mm
- net HRAM_DQ0: track 6.84 -> 20.1 mm
- net HRAM_CLK: track 7.61 -> 20.2 mm
- net HRAM_DQ3: track 7.60 -> 20.2 mm
- net DIR_JTDI: track 0.00 -> 12.6 mm
- net QSPI_IO1: track 6.52 -> 18.9 mm
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
Commit message: WIP
Parts:
- removed TP50, TP51, TP54, TP55, TP57, TP58, TP60, TP61, TP63, TP64, TP66, TP67, TP70, TP73, TP74, TP77, TP78, TP81, TP82, TP85, TP86, TP88, TP89, TP90, TP91, TP92: ~, TestPoint:TestPoint_Pad_D1.0mm
- C50, C51, C52, C53, C54, C55, C56, C57, C58, J5: moved to B.Cu
- moved U21 70.7 mm to (165.1, 70.4)
- moved J5 66.7 mm to (146.6, 93.3), turned to 90 degrees
- moved U20 62.8 mm to (165.1, 76.4)
- moved R67 59.4 mm to (176.2, 85.1)
- moved U17 59.4 mm to (174.2, 79.9)
- moved R66 59.4 mm to (176.2, 83.1)
- moved C71 59.4 mm to (178.2, 78.5)
- moved C72 59.4 mm to (178.2, 80.4)
- moved TP93 59.4 mm to (173.2, 83.6)
- moved U22 57.9 mm to (165.1, 64.4)
- moved U19 56.8 mm to (165.1, 82.4)
- moved J2 55.3 mm to (217.1, 85.3)
- moved R17 55.3 mm to (220.8, 84.0)
- moved R18 55.3 mm to (220.8, 86.0)
- moved R19 55.3 mm to (220.8, 88.0)
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Connections:
- R30 pad 1: Net-(U11-B1) -> Net-(U11-B3)
- R31 pad 1: Net-(U12-B1) -> Net-(U12-B3)
- R32 pad 1: Net-(U11-B2) -> Net-(U11-B4)
- R33 pad 1: Net-(U12-B2) -> Net-(U12-B4)
- R34 pad 1: Net-(U11-B3) -> Net-(U11-B1)
- R35 pad 1: Net-(U12-B3) -> Net-(U12-B1)
- R36 pad 1: Net-(U11-B4) -> Net-(U11-B2)
- R37 pad 1: Net-(U12-B4) -> Net-(U12-B2)
- R42 pad 1: Net-(U14-B1) -> Net-(U14-B3)
- R43 pad 1: Net-(U15-B1) -> Net-(U15-B3)
- R45 pad 1: Net-(U14-B2) -> Net-(U14-B4)
- R46 pad 1: Net-(U15-B2) -> Net-(U15-B4)
- R47 pad 1: Net-(U14-B3) -> Net-(U14-B1)
- R48 pad 1: Net-(U15-B3) -> Net-(U15-B1)
- R50 pad 1: Net-(U14-B4) -> Net-(U14-B2)
- R51 pad 1: Net-(U15-B4) -> Net-(U15-B2)
- U11 pad 1: DIR_JTCK -> DIR_JTDI
- U11 pad 2: DIR_JTMS -> GND
- U11 pad 3: DEBUG_JTCK -> DEBUG_JTDI
- U11 pad 4: DEBUG_JTMS -> DEBUG_JTDO
- U11 pad 5: DEBUG_JTDI -> DEBUG_JTCK
- U11 pad 6: DEBUG_JTDO -> DEBUG_JTMS
- U11 pad 7: DIR_JTDI -> DIR_JTCK
- U11 pad 8: GND -> DIR_JTMS
- U12 pad 1: GND -> SPARE_DIR4
- U12 pad 2: GND -> SPARE_DIR5
- U12 pad 3: TRACE_D3 -> SPARE_IO4
- U12 pad 4: TRACE_D2 -> SPARE_IO5
- U12 pad 5: SPARE_IO4 -> TRACE_D3
- U12 pad 6: SPARE_IO5 -> TRACE_D2
- U12 pad 7: SPARE_DIR4 -> GND
- U12 pad 8: SPARE_DIR5 -> GND
- U14 pad 2: DIR_NRST -> GND
- U14 pad 3: TRACE_CLK -> TRACE_D1
- U14 pad 4: DEBUG_NRST -> TRACE_D0
- U14 pad 5: TRACE_D1 -> TRACE_CLK
- U14 pad 6: TRACE_D0 -> DEBUG_NRST
- U14 pad 8: GND -> DIR_NRST
- U15 pad 1: SPARE_DIR2 -> SPARE_DIR0
- U15 pad 2: SPARE_DIR3 -> SPARE_DIR1
- U15 pad 3: SPARE_IO2 -> SPARE_IO0
- U15 pad 4: SPARE_IO3 -> SPARE_IO1
- U15 pad 5: SPARE_IO0 -> SPARE_IO2
- U15 pad 6: SPARE_IO1 -> SPARE_IO3
- U15 pad 7: SPARE_DIR0 -> SPARE_DIR2
- U15 pad 8: SPARE_DIR1 -> SPARE_DIR3
Routing:
- net DIR_JTDI: track 12.6 -> 1.39 mm, vias 0 -> 1
- net DEBUG_JTDI: track 11.3 -> 1.07 mm
- net DEBUG_JTDO: track 12.1 -> 1.94 mm
- net VT_DEBUG_JTDO: track 14.3 -> 5.16 mm
- net VTREF: track 20.3 -> 11.5 mm, vias 1 -> 2
- net DEBUG_JTMS: track 9.81 -> 1.03 mm
- net VT_DEBUG_JTCK: track 15.6 -> 7.05 mm
- net VT_DEBUG_JTMS: track 13.5 -> 5.16 mm
- net DEBUG_JTCK: track 9.88 -> 2.10 mm
- net HRAM_DQ0: track 20.1 -> 12.5 mm
- net DIR_JTMS: track 8.30 -> 0.87 mm
- net QSPI_SCK: track 18.9 -> 11.5 mm
- net HRAM_DQ1: track 20.2 -> 13.8 mm
- net HRAM_DQ4: track 20.2 -> 15.6 mm
- net HRAM_DQ3: track 20.2 -> 16.3 mm
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Other:
- outline, holes or cut-outs redrawn
- board text added: "CK"
- board text added: "CORTEX DEBUG 0.05{dblquote}"
- board text added: "DEBUG"
- board text added: "DI"
- board text added: "DO"
- board text added: "GND"
- board text added: "IO0"
- board text added: "IO1"
- board text added: "IO2"
- board text added: "IO3"
- board text added: "IO4"
- board text added: "IO5"
- board text added: "JTAG"
- board text added: "MS"
- board text added: "NC"
- board text added: "SPARE"
- board text added: "STATUS"
- board text added: "TRACE"
- board text added: "VTPWR"
- board text added: "VTREF"
- board text added: "Vref"
- board text added: "~{RST}"

Commit message: WIP
Parts:
- C59, C62, FB2, FB3, FB5: moved to B.Cu
- moved TP52 9.18 mm to (205.6, 66.7)
- moved FB5 8.76 mm to (204.8, 59.9)
- moved C62 7.35 mm to (202.1, 59.9)
- moved FB3 6.82 mm to (204.8, 64.4)
- moved FB2 5.56 mm to (204.8, 68.9)
- moved C59 3.55 mm to (202.1, 64.4)
- moved C54 2.99 mm to (202.1, 68.9), turned to 180 degrees
- moved C56 1.09 mm to (182.7, 79.5)
- moved C58 0.90 mm to (192.8, 79.5)
- moved C53 0.86 mm to (187.8, 79.5)
- moved C57 0.23 mm to (192.8, 82.1)
- moved C50 0.22 mm to (197.9, 82.1)
- moved C52 0.16 mm to (187.8, 82.1)
- moved C55 0.16 mm to (182.7, 82.1)
- moved C51 0.15 mm to (197.9, 79.5)
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Routing:
- net VTREF: track 11.5 -> 36.5 mm, vias 2 -> 4
- net GND: track 47.9 -> 71.7 mm, vias 27 -> 29
- net VT_DEBUG_JTDI: track 7.12 -> 29.6 mm
- net VT_DEBUG_JTDO: track 5.16 -> 26.9 mm
- net VT_DEBUG_JTCK: track 7.05 -> 28.1 mm
- net VT_DEBUG_NRST: track 5.16 -> 26.0 mm
- net VT_DEBUG_JTMS: track 5.16 -> 25.5 mm
- net DIR_JTMS: track 0.87 -> 15.3 mm
- net DEBUG_JTDO: track 1.94 -> 14.0 mm
- net DEBUG_JTDI: track 1.07 -> 13.0 mm
- net DIR_JTCK: track 2.00 -> 13.9 mm
- net DEBUG_JTMS: track 1.03 -> 12.9 mm
- net DEBUG_JTCK: track 2.10 -> 13.7 mm
- net DIR_NRST: track 2.33 -> 12.4 mm
- net DIR_JTDI: track 1.39 -> 10.3 mm, vias 1 -> 2
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- added copper zone on In1.Cu, net GND

Commit message: WIP
Parts:
- removed C67, C68, C69, C70: 100nF, Capacitor_SMD:C_0402_1005Metric
- removed J5: Conn_02x35_Odd_Even, Connector_Hirose_DF40:Hirose_DF40C-70DS-0.4V_2x35_P0.4mm
- C18, C43, C61, C63, C64, C65, C66, R21, R22, R23, R62, R63, R64, R65, TP32, TP36, TP40, TP44, TP48, TP93, TP94, TP95, TP96, TP97, TP98, TP99, U16, U7: moved to B.Cu
- moved TP99 79.7 mm to (165.1, 62.8), turned to 180 degrees
- moved TP98 74.2 mm to (165.1, 68.8), turned to 180 degrees
- moved TP97 69.4 mm to (165.1, 74.8), turned to 180 degrees
- moved TP96 68.4 mm to (165.1, 80.8), turned to 180 degrees
- moved TP95 64.0 mm to (165.1, 86.8), turned to 180 degrees
- moved TP94 61.5 mm to (165.1, 90.0), turned to 180 degrees
- moved R22 37.4 mm to (187.0, 97.8), turned to 180 degrees
- moved R23 36.8 mm to (186.9, 101.4), turned to 180 degrees
- moved R21 36.2 mm to (186.9, 100.0), turned to 180 degrees
- moved C18 33.7 mm to (187.0, 98.9), turned to 180 degrees
- moved TP48 28.4 mm to (183.8, 99.7), turned to 180 degrees
- moved R24 27.9 mm to (206.1, 88.9)
- moved R25 27.2 mm to (206.1, 89.9)
- moved R26 26.5 mm to (206.1, 90.9)
- moved R27 25.4 mm to (204.1, 88.9)
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Routing:
- net VT_SPARE_IO0: track 0.00 -> 26.7 mm
- net VT_SPARE_IO2: track 0.00 -> 26.6 mm
- net VT_SPARE_IO1: track 0.00 -> 26.6 mm
- net VT_SPARE_IO4: track 0.00 -> 26.6 mm
- net VT_SPARE_IO3: track 0.00 -> 26.6 mm
- net VT_SPARE_IO5: track 0.00 -> 26.6 mm
- net LED_DATA: track 0.54 -> 23.9 mm, vias 1 -> 2
- net JTDO: track 0.57 -> 18.7 mm
- net JTCK: track 0.59 -> 18.1 mm
- net JTDI: track 0.52 -> 17.4 mm
- net JTMS: track 0.59 -> 17.1 mm
- net HRAM_DQ4: track 15.6 -> 3.00 mm
- net LED_START: track 0.00 -> 11.9 mm, vias 0 -> 1
- net +5V: track 4.39 -> 15.6 mm, vias 1 -> 6
- net GND: track 71.7 -> 81.2 mm, vias 29 -> 34
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